Commit message: mrp face renders on ohmni robot in gazebo

File: ros_ws/src/tb_sim/tb_description/urdf/tb_sim.urdf.xacro (robot description, xacro)
@@ -187,11 +187,11 @@
       <origin xyz="0 0 0" rpy="0 0 0" />
       <geometry>
-        <mesh filename="package://tb_description/meshes/display_link.STL" />
-      </geometry>
-    </visual>
-    <collision>
-      <origin xyz="0 0 0" rpy="0 0 0" />
-      <geometry>
-        <mesh filename="package://tb_description/meshes/display_link.STL" />
+        <mesh filename="package://tb_description/meshes/display_link.dae" />
+      </geometry>
+    </visual>
+    <collision>
+      <origin xyz="0 0 0" rpy="0 0 0" />
+      <geometry>
+        <mesh filename="package://tb_description/meshes/display_link.dae" />
       </geometry>
     </collision>
